Commit message: fraksergo

File: scane/models/drone.urdf (robot description, URDF)
Before this commit: robot drone, 1 links, 0 joints
Links:
- link base_link: geometry collision mesh filename=modelfiles/mq9model.obj scale=0.2 0.2 0.2; visual mesh filename=modelfiles/mq9model.obj scale=0.2 0.2 0.2

File: scane/models/real_map.urdf (robot description, URDF)
Before this commit: robot real_map, 1 links, 0 joints
Links:
- link base_link: geometry collision mesh filename=modelfiles/real-3.obj scale=1 1 1; visual mesh filename=modelfiles/real-3.obj scale=1 1 1
