Commit message: frer

File: scane/models/real_map.urdf (robot description, URDF)
Before this commit: robot real_map, 1 links, 0 joints
Links:
- link base_link: geometry collision mesh filename=modelfiles/real-2.obj scale=1 1 1; visual mesh filename=modelfiles/real-2.obj scale=1 1 1

Commit message: falan map

File: scane/models/real_map.urdf (robot description, URDF)
Before this commit: robot real_map, 1 links, 0 joints
Links:
- link base_link: geometry collision mesh filename=modelfiles/Untitled.dae scale=1 1 1; visual mesh filename=modelfiles/Untitled.dae scale=1 1 1

Commit message: hukl

File: scane/models/real_map.urdf (robot description, URDF)
Before this commit: robot real_map, 1 links, 0 joints
Links:
- link base_link: geometry collision mesh filename=modelfiles/real-3.obj scale=0.01 0.01 0.01; visual mesh filename=modelfiles/real-3.obj scale=0.01 0.01 0.01
